File: aansturing lamp pcb/_autosave-aansturing lamp pcb.kicad_sch (KiCad schematic)
At the start: 20 parts, among them J1 Conn_01x07_Pin, U2 MCP16311MS, U3 INA169, U4 AD5245BRJZ50-RL7

Commit message: ok
Connections:
- net scl: now also J1.4 (Pin_4); no longer J1.5 (Pin_5)
- net sda: now also J1.5 (Pin_5); no longer J1.4 (Pin_4)
Changed lines of the file:
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@@
     (effects (font (size 1.27 1.27)) (justify right bottom))
   )
-  (label "sda" (at 37.465 38.1 180) (fields_autoplaced)
+  (label "scl" (at 37.465 38.1 180) (fields_autoplaced)
     (effects (font (size 1.27 1.27)) (justify right bottom))
   )
@@
     (effects (font (size 1.27 1.27)) (justify left bottom))
   )
-  (label "scl" (at 37.465 40.64 180) (fields_autoplaced)
+  (label "sda" (at 37.465 40.64 180) (fields_autoplaced)
     (effects (font (size 1.27 1.27)) (justify right bottom))
   )
