File: aansturing lamp pcb/aansturing lamp pcb.kicad_pcb (KiCad board)
At the start: 2 copper layers, 35 x 23 mm, 16 parts, among them J4 Conn_01x06_Pin, U1 LM317_SOT-223

Commit message: ok
Parts:
- moved C4 0.76 mm to (94.0, 84.3)
- moved H2 0.23 mm to (110.9, 91.9)
Routing:
- net /led+: track 29.8 -> 30.5 mm
Changed lines of the file:
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@@
   )
   (footprint "MountingHole:MountingHole_2.5mm" (layer "F.Cu")
-    (at 110.998 91.694)
+    (at 110.9 91.9)
     (descr "Mounting Hole 2.5mm, no annular")
     (tags "mounting hole 2.5mm no annular")
@@
     (property "ki_keywords" "mounting hole")
     (attr exclude_from_pos_files)
-    (fp_text reference "H2" (at -3.808 0.154) (layer "F.SilkS")
+    (fp_text reference "H2" (at -3.966 0.154) (layer "F.SilkS")
         (effects (font (size 1 1) (thickness 0.15)))
     )
@@
     (fp_circle (center 0 0) (end 2.75 0)
       (stroke (width 0.05) (type solid)) (fill none) (layer "F.CrtYd"))
-    (pad "" np_thru_hole circle (at 0 0) (size 2.5 2.5) (drill 2.5) (layers "*.Cu" "*.Mask"))
+    (pad "" np_thru_hole circle (at -0.1 0) (size 2.5 2.5) (drill 2.5) (layers "F&B.Cu" "*.Mask"))
   )
   (footprint "Capacitor_SMD:C_0805_2012Metric_Pad1.18x1.45mm_HandSolder" (layer "F.Cu")
-    (at 94.742 84.328 180)
+    (at 93.98 84.328 180)
     (descr "Capacitor SMD 0805 (2012 Metric), square (rectangular) end terminal, IPC_7351 nominal with elongated pad for handsoldering. (Body size source: IPC-SM-782 page 76, https://www.pcb-3d.com/wordpress/wp-content/uploads/ipc-sm-782a_amendment_1_and_2.pdf, https://docs.google.com/spreadsheets/d/1BsfQQcO9C6DZCsRaXUlFlo91Tg2WpOkGARC1WS5S8t0/edit?usp=sharing), generated with kicad-footprint-generator")
     (tags "capacitor handsolder")
@@
     (property "ki_keywords" "capacitor cap")
     (attr smd)
-    (fp_text reference "C4" (at 0 -1.68) (layer "F.SilkS")
+    (fp_text reference "C4" (at -2.794 -1.27) (layer "F.SilkS")
         (effects (font (size 1 1) (thickness 0.15)))
     )
@@
     (property "ki_keywords" "capacitor cap")
     (attr smd)
-    (fp_text reference "C1" (at 0.0872 1.8924 90) (layer "F.SilkS")
+    (fp_text reference "C1" (at 0.254 -1.778 90) (layer "F.SilkS")
         (effects (font (size 1 1) (thickness 0.15)))
     )
@@
   (segment (start 94.319996 77.978) (end 94.234 78.063996) (width 0.5) (layer "F.Cu") (net 8))
   (segment (start 97.268 73.8225) (end 97.9385 73.152) (width 0.5) (layer "F.Cu") (net 8))
+  (segment (start 95.9315 83.414) (end 95.0175 84.328) (width 0.5) (layer "F.Cu") (net 9))
+  (segment (start 99.568 83.414) (end 95.9315 83.414) (width 0.5) (layer "F.Cu") (net 9))
   (segment (start 101.6 85.09) (end 101.6 87.376) (width 0.5) (layer "F.Cu") (net 9))
   (segment (start 99.568 73.422) (end 99.838 73.152) (width 0.5) (layer "F.Cu") (net 9))
   (segment (start 99.568 83.414) (end 99.924 83.414) (width 0.5) (layer "F.Cu") (net 9))
-  (segment (start 96.6935 83.414) (end 95.7795 84.328) (width 0.5) (layer "F.Cu") (net 9))
   (segment (start 99.568 77.114) (end 99.568 73.422) (width 0.5) (layer "F.Cu") (net 9))
   (segment (start 99.568 77.114) (end 99.568 83.414) (width 0.5) (layer "F.Cu") (net 9))
-  (segment (start 99.568 83.414) (end 96.6935 83.414) (width 0.5) (layer "F.Cu") (net 9))
   (segment (start 102.13 80.852) (end 99.568 83.414) (width 0.5) (layer "F.Cu") (net 9))
   (segment (start 99.924 83.414) (end 101.6 85.09) (width 0.5) (layer "F.Cu") (net 9))

Commit message: ok
Parts:
- removed C1: 1nF, Capacitor_SMD:C_0805_2012Metric_Pad1.18x1.45mm_HandSolder
- removed C2: 0.01µF, Capacitor_SMD:C_0805_2012Metric_Pad1.18x1.45mm_HandSolder
- removed C3: 0.1µF, Capacitor_SMD:C_0805_2012Metric_Pad1.18x1.45mm_HandSolder
- removed C4: 1µF, Capacitor_SMD:C_0805_2012Metric_Pad1.18x1.45mm_HandSolder
- removed J4: Conn_01x06_Pin, Connector_PinHeader_2.54mm:PinHeader_1x06_P2.54mm_Vertical
- removed R4: 1k, Resistor_SMD:R_0805_2012Metric_Pad1.20x1.40mm_HandSolder
- removed Tled+1: led+, TestPoint:TestPoint_Pad_1.5x1.5mm
- removed U1: LM317_SOT-223, Package_TO_SOT_SMD:SOT-223-3_TabPin2
- removed currentsensor1: ACS712xLCTR-20A, Package_SO:SOIC-8_3.9x4.9mm_P1.27mm
- added C6: C_boost, Capacitor_SMD:C_0805_2012Metric_Pad1.18x1.45mm_HandSolder, F.Cu at (101.9, 87.7)
- added C7: C_Small, Capacitor_SMD:C_0805_2012Metric_Pad1.18x1.45mm_HandSolder, F.Cu at (98.3, 74.1)
- added C8: Cvcc, Capacitor_SMD:C_0805_2012Metric_Pad1.18x1.45mm_HandSolder, F.Cu at (101.7, 74.3)
- added C9: C_out, Capacitor_SMD:C_0805_2012Metric_Pad1.18x1.45mm_HandSolder, F.Cu at (89.3, 89.8)
- added J1: Conn_01x07_Pin, Connector_PinHeader_2.54mm:PinHeader_1x07_P2.54mm_Vertical, B.Cu at (82.0, 75.4)
- added L2: L_Small, Inductor_SMD:L_0805_2012Metric_Pad1.05x1.20mm_HandSolder, F.Cu at (100.9, 91.1)
- added R1: Rs, Resistor_SMD:R_0805_2012Metric_Pad1.20x1.40mm_HandSolder, F.Cu at (98.6, 88.8)
- added R2: R_en, Resistor_SMD:R_0805_2012Metric_Pad1.20x1.40mm_HandSolder, F.Cu at (98.3, 77.1)
- added R5: Rb, Resistor_SMD:R_0805_2012Metric_Pad1.20x1.40mm_HandSolder, F.Cu at (96.3, 82.6)
- added R7: Rl, Resistor_SMD:R_0805_2012Metric_Pad1.20x1.40mm_HandSolder, F.Cu at (89.4, 87.8)
- added U2: MCP16311MS, Package_SO:MSOP-8_3x3mm_P0.65mm, F.Cu at (101.6, 82.3)
- added U3: INA169, Package_TO_SOT_SMD:SOT-23-5, F.Cu at (93.9, 88.8)
- added U4: AD5245BRJZ50-RL7, own-footprints:SOT65P280X145-8N, F.Cu at (91.3, 81.7)
- R3: value 220 -> R50K
- moved R3 17.1 mm to (87.0, 83.2), turned to 90 degrees
- moved Tenable1 13.4 mm to (106.2, 75.5)
- moved Tground1 6.78 mm to (90.3, 92.5)
- moved mosfet1 1.37 mm to (90.8, 75.5)
Connections:
- R3 pad 1: Net-(U1-ADJ) -> /stroom+
- R3 pad 2: /led+ -> /R_{digin}
- led1 pad 1: /led- -> GND
Routing:
- net /led+: track 30.5 -> 0.00 mm
- net +5V: track 20.9 -> 0.00 mm
- net +12V: track 15.1 -> 0.00 mm
- net /led-: track 14.6 -> 0.00 mm
- net /A_{0}: track 12.8 -> 0.00 mm
- net /I/0_{0}: track 7.59 -> 0.00 mm
- net Net-(U1-ADJ): track 6.69 -> 0.00 mm
- net /enable: track 11.1 -> 4.96 mm
- net Net-(U2-Vcc): track 0.00 -> 4.87 mm
- net Net-(U2-EN): track 0.00 -> 3.87 mm
- net Net-(currentsensor1-FILTER): track 3.34 -> 0.00 mm
- net GND: track 3.21 -> 0.00 mm, vias 1 -> 0
- net Net-(U2-SW): track 0.00 -> 2.35 mm

Commit message: ok
Parts:
- moved Tenable1 9.58 mm to (97.8, 80.1)
- moved R3 9.09 mm to (89.3, 91.9), turned to 180 degrees
- moved Tground1 4.97 mm to (85.3, 92.2)
- moved L2 3.75 mm to (98.0, 88.6)
- moved R1 2.86 mm to (98.0, 91.6), turned to -90 degrees
- moved R5 2.20 mm to (94.9, 84.3)
- moved U4 2.02 mm to (90.3, 83.4)
- moved C6 0.91 mm to (102.0, 88.6), turned to 0 degrees
- moved mosfet1 0.29 mm to (90.9, 75.7)
Routing:
- net +3.3V: track 0.00 -> 27.9 mm
- net /led+: track 0.00 -> 23.3 mm
- net /stroom+: track 0.00 -> 18.4 mm
- net /ad0: track 0.00 -> 17.3 mm
- net +12V: track 0.00 -> 15.5 mm
- net GND: track 0.00 -> 14.1 mm, vias 0 -> 4
- net /I/0_{0}: track 0.00 -> 11.3 mm
- net /scl: track 0.00 -> 10.8 mm
- net /R_{digin}: track 0.00 -> 10.7 mm
- net /enable: track 4.96 -> 13.5 mm
- net /sda: track 0.00 -> 8.38 mm
- net Net-(U2-BOOST): track 0.00 -> 4.71 mm
- net /R_{digout}: track 0.00 -> 2.42 mm
- net Net-(U2-SW): track 2.35 -> 4.37 mm

Commit message: ok
Parts:
- moved J1 0.41 mm to (82.0, 75.8)
Routing:
- net +12V: track 15.5 -> 0.00 mm
- net /ad0: track 17.3 -> 2.40 mm
- net +3.3V: track 27.9 -> 13.7 mm
- net /I/0_{0}: track 11.3 -> 0.00 mm
- net /scl: track 10.8 -> 0.00 mm
- net /sda: track 8.38 -> 0.00 mm
Changed lines of the file:
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@@
   )
   (footprint "Connector_PinHeader_2.54mm:PinHeader_1x07_P2.54mm_Vertical" (layer "B.Cu")
-    (at 82.042 75.438 180)
+    (at 82 75.85 180)
     (descr "Through hole straight pin header, 1x07, 2.54mm pitch, single row")
     (tags "Through hole pin header THT 1x07 2.54mm single row")
@@
   (segment (start 101.895 87.5225) (end 101.895 84.4025) (width 0.25) (layer "F.Cu") (net 3))
   (segment (start 103.0185 88.646) (end 101.895 87.5225) (width 0.25) (layer "F.Cu") (net 3))
-  (segment (start 84.091996 76.708) (end 86.377996 74.422) (width 0.25) (layer "F.Cu") (net 4))
-  (segment (start 81.153 76.708) (end 84.091996 76.708) (width 0.25) (layer "F.Cu") (net 4))
-  (segment (start 86.377996 74.422) (end 86.781996 74.422) (width 0.25) (layer "F.Cu") (net 4))
-  (segment (start 82.042 80.518) (end 80.518 78.994) (width 0.25) (layer "F.Cu") (net 4))
-  (segment (start 80.518 78.994) (end 80.518 77.343) (width 0.25) (layer "F.Cu") (net 4))
-  (segment (start 80.518 77.343) (end 81.153 76.708) (width 0.25) (layer "F.Cu") (net 4))
   (segment (start 101.895 75.5725) (end 101.895 80.1775) (width 0.25) (layer "F.Cu") (net 5))
   (segment (start 101.71 75.3875) (end 101.895 75.5725) (width 0.25) (layer "F.Cu") (net 5))
-  (segment (start 93.430996 72.771) (end 95.081996 74.422) (width 0.25) (layer "F.Cu") (net 6))
-  (segment (start 83.566 72.771) (end 93.430996 72.771) (width 0.25) (layer "F.Cu") (net 6))
-  (segment (start 82.042 74.295) (end 83.566 72.771) (width 0.25) (layer "F.Cu") (net 6))
-  (segment (start 82.042 75.438) (end 82.042 74.295) (width 0.25) (layer "F.Cu") (net 6))
   (segment (start 96.894 88.646) (end 94.230751 88.646) (width 0.25) (layer "F.Cu") (net 7))
   (segment (start 93.116751 89.76) (end 92.7325 89.76) (width 0.25) (layer "F.Cu") (net 7))
@@
   (segment (start 105.711 80.852) (end 108.712 80.852) (width 0.25) (layer "F.Cu") (net 9))
   (segment (start 96.266 82.042) (end 93.726 82.042) (width 0.25) (layer "F.Cu") (net 10))
-  (segment (start 93.726 82.042) (end 93.726 80.518) (width 0.25) (layer "F.Cu") (net 10))
   (segment (start 97.917 85.217) (end 97.917 83.693) (width 0.25) (layer "F.Cu") (net 10))
   (segment (start 96.901 86.233) (end 97.917 85.217) (width 0.25) (layer "F.Cu") (net 10))
   (segment (start 95.0075 87.86) (end 96.6345 86.233) (width 0.25) (layer "F.Cu") (net 10))
   (segment (start 93.726 82.5206) (end 93.726 82.042) (width 0.25) (layer "F.Cu") (net 10))
-  (segment (start 92.202 78.994) (end 83.058 78.994) (width 0.25) (layer "F.Cu") (net 10))
   (segment (start 92.4774 83.7692) (end 93.726 82.5206) (width 0.25) (layer "F.Cu") (net 10))
   (segment (start 96.6345 86.233) (end 96.901 86.233) (width 0.25) (layer "F.Cu") (net 10))
-  (segment (start 93.726 80.518) (end 92.202 78.994) (width 0.25) (layer "F.Cu") (net 10))
   (segment (start 91.4654 83.7692) (end 92.4774 83.7692) (width 0.25) (layer "F.Cu") (net 10))
-  (segment (start 83.058 78.994) (end 82.042 77.978) (width 0.25) (layer "F.Cu") (net 10))
   (segment (start 97.917 83.693) (end 96.266 82.042) (width 0.25) (layer "F.Cu") (net 10))
-  (segment (start 89.1286 82.4738) (end 85.1662 82.4738) (width 0.25) (layer "F.Cu") (net 11))
-  (segment (start 85.1662 82.4738) (end 82.042 85.598) (width 0.25) (layer "F.Cu") (net 11))
-  (segment (start 91.4654 82.4738) (end 91.4654 81.9404) (width 0.25) (layer "F.Cu") (net 12))
-  (segment (start 91.4654 81.9404) (end 91.059 81.534) (width 0.25) (layer "F.Cu") (net 12))
-  (segment (start 91.059 81.534) (end 83.566 81.534) (width 0.25) (layer "F.Cu") (net 12))
-  (segment (start 83.566 81.534) (end 82.042 83.058) (width 0.25) (layer "F.Cu") (net 12))
-  (segment (start 87.0712 83.1088) (end 82.042 88.138) (width 0.25) (layer "F.Cu") (net 13))
   (segment (start 90.36 87.79) (end 92.6625 87.79) (width 0.25) (layer "F.Cu") (net 13))
-  (segment (start 90.36 87.79) (end 90.36 83.3727) (width 0.25) (layer "F.Cu") (net 13))
   (segment (start 92.6625 87.79) (end 92.7325 87.86) (width 0.25) (layer "F.Cu") (net 13))
-  (segment (start 90.36 83.3727) (end 90.0961 83.1088) (width 0.25) (layer "F.Cu") (net 13))
-  (segment (start 90.0961 83.1088) (end 89.1286 83.1088) (width 0.25) (layer "F.Cu") (net 13))
-  (segment (start 89.1286 83.1088) (end 87.0712 83.1088) (width 0.25) (layer "F.Cu") (net 13))
   (segment (start 99.34 77.1) (end 99.34 77.508959) (width 0.25) (layer "F.Cu") (net 14))
   (segment (start 101.245 79.413959) (end 101.245 80.1775) (width 0.25) (layer "F.Cu") (net 14))
