File: testboard AL5801/testboard AL5801.kicad_pcb (KiCad board)
At the start: 2 copper layers, 35 x 23 mm, 14 parts, among them J1 Conn_01x07_Pin, J2 Conn_01x02_Pin, U1 AL5801W6-7, U2 INA169

Commit message: pcbs al580 en stcs05
Parts:
- removed J2: Conn_01x02_Pin, Connector_PinSocket_2.54mm:PinSocket_1x02_P2.54mm_Vertical
- added J3: Screw_Terminal_01x02, TerminalBlock_Phoenix:TerminalBlock_Phoenix_PT-1,5-2-5.0-H_1x02_P5.00mm_Horizontal, F.Cu at (155.8, 72.1)
- J1: moved to B.Cu
- moved R1 42.9 mm to (148.4, 68.4), turned to 90 degrees
- moved U1 42.5 mm to (147.2, 63.2), turned to 180 degrees
- moved R3 37.4 mm to (143.8, 63.3), turned to -90 degrees
- moved R4 36.7 mm to (142.9, 72.2), turned to 180 degrees
- moved JP1 35.7 mm to (149.0, 59.7)
- moved R2 34.2 mm to (140.6, 63.3), turned to -90 degrees
- moved JP2 32.9 mm to (148.4, 72.9), turned to -90 degrees
- moved R5 28.6 mm to (135.0, 73.7)
- moved U2 3.37 mm to (142.8, 68.0)
- moved mosfet1 2.22 mm to (135.5, 63.9), turned to 180 degrees
- turned J1 to 180 degrees
Connections:
- R1 pad 1: /led- -> /led+
- U1 pad 3: /enable -> /led-
- U2 pad 5: +3.3V -> +3V3
Routing:
- net /led+: track 0.00 -> 41.7 mm, vias 0 -> 1
- net /led-: track 0.00 -> 18.9 mm
- net /ad0: track 0.00 -> 18.8 mm
- net +3V3: track 0.00 -> 16.3 mm
- net /enable: track 0.00 -> 11.6 mm
- net Net-(U1-FB): track 0.00 -> 8.17 mm
- net VSS: track 0.00 -> 6.62 mm
- net /I/O: track 0.00 -> 5.99 mm
- net /enable : track 0.00 -> 3.41 mm
- net Net-(U1-BIAS): track 0.00 -> 3.21 mm
- added copper zone on F.Cu, net GND
Other:
- board text added: "12V 3..3V I/O SCL SDA ad0 GND"
