File: testboard AL5801/testboard AL5801.kicad_sch (KiCad schematic)
At the start: 14 parts, among them J1 Conn_01x07_Pin, J2 Conn_01x02_Pin, U1 AL5801W6-7, U2 INA169

Commit message: pcbs al580 en stcs05
Parts:
- removed J2: Conn_01x02_Pin, Connector_PinSocket_2.54mm:PinSocket_1x02_P2.54mm_Vertical, symbol Connector:Conn_01x02_Pin
- added J3: Screw_Terminal_01x02, TerminalBlock_Phoenix:TerminalBlock_Phoenix_PT-1,5-2-5.0-H_1x02_P5.00mm_Horizontal, symbol Connector:Screw_Terminal_01x02
Connections:
- net +3.3V is gone; now on net +3V3: U2.5 (V+)
- net enable: no longer U1.3 (OUT)
- net led+: now also R1.1, J3.1 (Pin_1)
- net led-: now also U1.3 (OUT), J3.2 (Pin_2); no longer R1.1
Changed lines of the file:
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@@
     (stroke (width 0) (type default))
   )
-  (label "enable" (at 88.265 79.375 0) (fields_autoplaced)
+  (label "led-" (at 88.265 79.375 0) (fields_autoplaced)
     (effects (font (size 1.27 1.27)) (justify left bottom))
   )
@@
     (effects (font (size 1.27 1.27)) (justify left bottom))
   )
-  (label "led-" (at 72.39 74.295 0) (fields_autoplaced)
-    (effects (font (size 1.27 1.27)) (justify left bottom))
-  )
-  (symbol (lib_id "Connector:Conn_01x02_Pin") (at 125.73 46.355 180) (unit 1)
-    (in_bom yes) (on_board yes) (dnp no) (fields_autoplaced)
-    (property "Reference" "J2" (at 127 44.45 0)
-      (effects (font (size 1.27 1.27)) (justify right))
-    )
-    (property "Value" "Conn_01x02_Pin" (at 127 46.99 0)
-      (effects (font (size 1.27 1.27)) (justify right))
-    )
-    (property "Footprint" "Connector_PinSocket_2.54mm:PinSocket_1x02_P2.54mm_Vertical" (at 125.73 46.355 0)
-      (effects (font (size 1.27 1.27)) hide)
-    )
-    (property "Datasheet" "~" (at 125.73 46.355 0)
-      (effects (font (size 1.27 1.27)) hide)
-    )
-    (pin "1")
-    (pin "2")
-    (instances
-      (project "testboard AL5801"
-        (path "/22d3873b-424a-4842-bcc7-1f3288cc1bd6"
-          (reference "J2") (unit 1)
-        )
-      )
-    )
+  (label "led+" (at 72.39 74.295 0) (fields_autoplaced)
+    (effects (font (size 1.27 1.27)) (justify left bottom))
   )
   (symbol (lib_id "Jumper:SolderJumper_2_Open") (at 56.515 67.31 0) (unit 1)
@@
     )
   )
-  (symbol (lib_id "power:+3.3V") (at 86.995 34.925 0) (unit 1)
+  (symbol (lib_id "power:+3V3") (at 86.995 34.925 0) (unit 1)
     (in_bom yes) (on_board yes) (dnp no) (fields_autoplaced)
     (property "Reference" "#PWR02" (at 86.995 38.735 0)
       (effects (font (size 1.27 1.27)) hide)
     )
-    (property "Value" "+3.3V" (at 86.995 31.75 0)
+    (property "Value" "+3V3" (at 86.995 31.115 0)
       (effects (font (size 1.27 1.27)))
     )
@@
         (path "/22d3873b-424a-4842-bcc7-1f3288cc1bd6"
           (reference "#PWR02") (unit 1)
-        )
-      )
-      (project "aansturing lamp pcb"
-        (path "/c70ffad9-435e-456d-9ee7-1dbdfd774131"
-          (reference "#PWR015") (unit 1)
         )
       )
@@
         )
       )
+    )
+  )
+  (symbol (lib_id "Connector:Screw_Terminal_01x02") (at 125.73 43.815 0) (unit 1)
+    (in_bom yes) (on_board yes) (dnp no) (fields_autoplaced)
+    (property "Reference" "J3" (at 128.905 44.45 0)
+      (effects (font (size 1.27 1.27)) (justify left))
+    )
+    (property "Value" "Screw_Terminal_01x02" (at 128.905 46.99 0)
+      (effects (font (size 1.27 1.27)) (justify left))
+    )
+    (property "Footprint" "TerminalBlock_Phoenix:TerminalBlock_Phoenix_PT-1,5-2-5.0-H_1x02_P5.00mm_Horizontal" (at 125.73 43.815 0)
+      (effects (font (size 1.27 1.27)) hide)
+    )
+    (property "Datasheet" "~" (at 125.73 43.815 0)
+      (effects (font (size 1.27 1.27)) hide)
+    )
+    (pin "1")
+    (pin "2")
+    (instances
+      (project "testboard AL5801"
+        (path "/22d3873b-424a-4842-bcc7-1f3288cc1bd6"
+          (reference "J3") (unit 1)
+        )
+      )
