File: stcs05/stcs05.kicad_sch (KiCad schematic)
At the start: 14 parts, among them J1 Conn_01x07_Pin, J3 Screw_Terminal_01x02, U1 STCS05DR, U2 INA169

Commit message: aanpassingen
Parts:
- R4: footprint Resistor_SMD:R_0805_2012Metric_Pad1.20x1.40mm_HandSolder -> Resistor_SMD:R_2512_6332Metric_Pad1.40x3.35mm_HandSolder
Changed lines of the file:
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@@
       (effects (font (size 1.27 1.27)) (justify right))
     )
-    (property "Footprint" "Resistor_SMD:R_0805_2012Metric_Pad1.20x1.40mm_HandSolder" (at 72.39 41.275 0)
+    (property "Footprint" "Resistor_SMD:R_2512_6332Metric_Pad1.40x3.35mm_HandSolder" (at 72.39 41.275 0)
       (effects (font (size 1.27 1.27)) hide)
     )

Commit message: ok
Parts:
- added R5: 470R, Resistor_SMD:R_0805_2012Metric_Pad1.20x1.40mm_HandSolder, symbol Device:R_Small
- C1: value C_Small -> 0.1µF
- C2: value C_Small -> 0.47µF
- R5: value Rl -> 3k3
- R5: value Rl -> 1R_sense
- R5: value Rl -> 100R
Connections:
- net GND: now also R5.1
- net I/O: now also R5.2
Changed lines of the file:
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@@
   (junction (at 72.39 38.735) (diameter 0) (color 0 0 0 0)
   )
+  (junction (at 104.775 59.69) (diameter 0) (color 0 0 0 0)
+  )
   (junction (at 131.445 40.64) (diameter 0) (color 0 0 0 0)
   )
@@
     (stroke (width 0) (type default))
   )
+  (wire (pts (xy 104.775 59.69) (xy 111.125 59.69))
+    (stroke (width 0) (type default))
+  )
   (wire (pts (xy 144.145 78.74) (xy 144.145 80.645))
     (stroke (width 0) (type default))
@@
     (stroke (width 0) (type default))
   )
+  (wire (pts (xy 104.775 68.58) (xy 104.775 66.675))
+    (stroke (width 0) (type default))
+  )
   (wire (pts (xy 72.39 43.815) (xy 74.295 43.815))
     (stroke (width 0) (type default))
@@
     (stroke (width 0) (type default))
   )
+  (wire (pts (xy 104.775 61.595) (xy 104.775 59.69))
+    (stroke (width 0) (type default))
+  )
   (wire (pts (xy 144.145 67.945) (xy 144.145 73.66))
     (stroke (width 0) (type default))
@@
     (stroke (width 0) (type default))
   )
-  (wire (pts (xy 107.315 59.69) (xy 111.125 59.69))
+  (wire (pts (xy 97.79 59.69) (xy 104.775 59.69))
     (stroke (width 0) (type default))
   )
@@
     (effects (font (size 1.27 1.27)) (justify right bottom))
   )
-  (label "I{slash}O" (at 107.315 59.69 0) (fields_autoplaced)
+  (label "I{slash}O" (at 97.79 59.69 0) (fields_autoplaced)
     (effects (font (size 1.27 1.27)) (justify left bottom))
   )
@@
   )
   (symbol (lib_id "Connector:Screw_Terminal_01x02") (at 200.66 57.785 0) (unit 1)
-    (in_bom yes) (on_board yes) (dnp no) (fields_autoplaced)
+    (in_bom yes) (on_board yes) (dnp no)
     (property "Reference" "J3" (at 203.835 58.42 0)
       (effects (font (size 1.27 1.27)) (justify left))
@@
     )
   )
-  (symbol (lib_id "power:GND") (at 79.375 52.705 0) (unit 1)
-    (in_bom yes) (on_board yes) (dnp no) (fields_autoplaced)
-    (property "Reference" "#PWR09" (at 79.375 59.055 0)
-      (effects (font (size 1.27 1.27)) hide)
-    )
-    (property "Value" "GND" (at 81.915 53.9749 0)
+  (symbol (lib_id "power:GND") (at 104.775 68.58 0) (unit 1)
+    (in_bom yes) (on_board yes) (dnp no) (fields_autoplaced)
+    (property "Reference" "#PWR09" (at 104.775 74.93 0)
+      (effects (font (size 1.27 1.27)) hide)
+    )
+    (property "Value" "GND" (at 107.315 69.8499 0)
       (effects (font (size 1.27 1.27)) (justify left))
     )
-    (property "Footprint" "" (at 79.375 52.705 0)
-      (effects (font (size 1.27 1.27)) hide)
-    )
-    (property "Datasheet" "" (at 79.375 52.705 0)
+    (property "Footprint" "" (at 104.775 68.58 0)
+      (effects (font (size 1.27 1.27)) hide)
+    )
+    (property "Datasheet" "" (at 104.775 68.58 0)
       (effects (font (size 1.27 1.27)) hide)
     )
@@
       (project "stcs05"
         (path "/ee2c9ab2-da3b-4785-b37f-83a0ffb53302"
+          (reference "#PWR015") (unit 1)
+        )
+      )
+    )
+  )
+  (symbol (lib_id "power:GND") (at 79.375 52.705 0) (unit 1)
+    (in_bom yes) (on_board yes) (dnp no) (fields_autoplaced)
+    (property "Reference" "#PWR09" (at 79.375 59.055 0)
+      (effects (font (size 1.27 1.27)) hide)
+    )
+    (property "Value" "GND" (at 81.915 53.9749 0)
+      (effects (font (size 1.27 1.27)) (justify left))
+    )
+    (property "Footprint" "" (at 79.375 52.705 0)
+      (effects (font (size 1.27 1.27)) hide)
+    )
+    (property "Datasheet" "" (at 79.375 52.705 0)
+      (effects (font (size 1.27 1.27)) hide)
+    )
+    (pin "1")
+    (instances
+      (project "testboard AL5801"
+        (path "/22d3873b-424a-4842-bcc7-1f3288cc1bd6"
+          (reference "#PWR09") (unit 1)
+        )
+      )
+      (project "aansturing lamp pcb"
+        (path "/c70ffad9-435e-456d-9ee7-1dbdfd774131"
+          (reference "#PWR011") (unit 1)
+        )
+      )
+      (project "stcs05"
+        (path "/ee2c9ab2-da3b-4785-b37f-83a0ffb53302"
           (reference "#PWR07") (unit 1)
         )
@@
       (effects (font (size 1.27 1.27)))
     )
-    (property "Value" "C_Small" (at 138.4363 38.1 90)
+    (property "Value" "0.1µF" (at 138.4363 38.1 90)
       (effects (font (size 1.27 1.27)))
     )
@@
       (effects (font (size 1.27 1.27)) (justify right))
     )
-    (property "Value" "Rl" (at 86.995 46.99 0)
+    (property "Value" "3k3" (at 85.725 47.625 0)
       (effects (font (size 1.27 1.27)) (justify right))
     )
@@
       (effects (font (size 1.27 1.27)) (justify right))
     )
-    (property "Value" "Rl" (at 132.715 78.105 0)
+    (property "Value" "1R_sense" (at 127 78.105 0)
       (effects (font (size 1.27 1.27)) (justify right))
     )
@@
       (effects (font (size 1.27 1.27)) (justify right))
     )
-    (property "Value" "C_Small" (at 153.67 76.835 0)
+    (property "Value" "0.47µF" (at 153.67 76.835 0)
       (effects (font (size 1.27 1.27)) (justify right))
     )
@@
     )
   )
+  (symbol (lib_id "Device:R_Small") (at 104.775 64.135 180) (unit 1)
+    (in_bom yes) (on_board yes) (dnp no)
+    (property "Reference" "R5" (at 100.33 63.5 0)
+      (effects (font (size 1.27 1.27)) (justify right))
+    )
+    (property "Value" "470R" (at 97.79 65.405 0)
+      (effects (font (size 1.27 1.27)) (justify right))
+    )
+    (property "Footprint" "Resistor_SMD:R_0805_2012Metric_Pad1.20x1.40mm_HandSolder" (at 104.775 64.135 0)
+      (effects (font (size 1.27 1.27)) hide)
+    )
+    (property "Datasheet" "~" (at 104.775 64.135 0)
+      (effects (font (size 1.27 1.27)) hide)
+    )
+    (pin "1")
+    (pin "2")
+    (instances
+      (project "stcs05"
+        (path "/ee2c9ab2-da3b-4785-b37f-83a0ffb53302"
+          (reference "R5") (unit 1)
+        )
+      )
+    )
+  )
   (symbol (lib_id "power:GND") (at 90.805 50.165 0) (unit 1)
     (in_bom yes) (on_board yes) (dnp no) (fields_autoplaced)
@@
       (effects (font (size 1.27 1.27)) (justify right))
     )
-    (property "Value" "Rl" (at 127.635 38.735 0)
-      (effects (font (size 1.27 1.27)) (justify right))
-    )
+    (property "Value" "100R" (at 125.095 38.735 0)
+      (effects (font (size 1.27 1.27)) (justify right))
+    )
