File: AL5801/testboard AL5801.kicad_pcb (KiCad board)
At the start: 2 copper layers, 35 x 23 mm, 14 parts, among them J1 Conn_01x07_Pin, J3 Screw_Terminal_01x02, U1 AL5801W6-7, U2 INA169

Commit message: aanpassingen
Parts:
- R4: footprint Resistor_SMD:R_0805_2012Metric_Pad1.20x1.40mm_HandSolder -> Resistor_SMD:R_2512_6332Metric_Pad1.40x3.35mm_HandSolder
- moved R4 4.17 mm to (142.8, 76.4)
Connections:
- R4 pad 2: /enable  -> /enable
- U2 pad 3: /enable  -> /enable
Routing:
- net /enable: track 11.6 -> 33.6 mm, vias 0 -> 2
- net /enable : track 3.41 -> 0.00 mm
- net /led+: track 41.7 -> 41.2 mm

Commit message: ok
Connections:
- net /enable renamed /V_{in+}
Other:
- board text added: "AL5801"
Changed lines of the file:
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@@
   (net 11 "/ad0")
   (net 12 "/led+")
-  (net 13 "/enable")
+  (net 13 "/V_{in+}")
   (footprint "MountingHole:MountingHole_2.5mm" (layer "F.Cu")
     (at 157.48 78.1812)
@@
       (stroke (width 0.05) (type solid)) (layer "F.CrtYd"))
     (pad "1" smd rect (at -0.65 0) (size 1 1.5) (layers "F.Cu" "F.Mask")
-      (net 13 "/enable") (pinfunction "A") (pintype "passive"))
+      (net 13 "/V_{in+}") (pinfunction "A") (pintype "passive"))
     (pad "2" smd rect (at 0.65 0) (size 1 1.5) (layers "F.Cu" "F.Mask")
       (net 12 "/led+") (pinfunction "B") (pintype "passive"))
@@
       (net 12 "/led+") (pintype "passive"))
     (pad "2" smd roundrect (at 3.05 0 180) (size 1.4 3.35) (layers "F.Cu" "F.Paste" "F.Mask") (roundrect_rratio 0.178571)
-      (net 13 "/enable") (pintype "passive"))
+      (net 13 "/V_{in+}") (pintype "passive"))
     (model "${KICAD6_3DMODEL_DIR}/Resistor_SMD.3dshapes/R_2512_6332Metric.wrl"
       (offset (xyz 0 0 0))
@@
       (net 2 "GND") (pinfunction "GND") (pintype "power_in"))
     (pad "3" smd roundrect (at -1.1375 0.95) (size 1.325 0.6) (layers "F.Cu" "F.Paste" "F.Mask") (roundrect_rratio 0.25)
-      (net 13 "/enable") (pinfunction "+") (pintype "input"))
+      (net 13 "/V_{in+}") (pinfunction "+") (pintype "input"))
     (pad "4" smd roundrect (at 1.1375 0.95) (size 1.325 0.6) (layers "F.Cu" "F.Paste" "F.Mask") (roundrect_rratio 0.25)
       (net 12 "/led+") (pinfunction "-") (pintype "input"))
@@
       (net 2 "GND") (pintype "passive") (thermal_bridge_angle 45))
     (pad "3" smd roundrect (at -1.27 4.149996 270) (size 1.9 1.5) (layers "F.Cu" "F.Paste" "F.Mask") (roundrect_rratio 0.25)
-      (net 13 "/enable") (pintype "passive") (thermal_bridge_angle 45))
+      (net 13 "/V_{in+}") (pintype "passive") (thermal_bridge_angle 45))
     (pad "4" smd roundrect (at 1.27 4.149996 270) (size 1.9 1.5) (layers "F.Cu" "F.Paste" "F.Mask") (roundrect_rratio 0.25)
       (net 1 "VSS") (pintype "passive") (thermal_bridge_angle 45))
@@
     (effects (font (size 1.5 1.5) (thickness 0.3) bold) (justify left bottom mirror))
   )
+  (gr_text "AL5801" (at 140.843 81.026) (layer "F.SilkS")
+    (effects (font (size 1 1) (thickness 0.15)) (justify left bottom))
+  )
   (segment (start 131.613955 62.145) (end 128.575 62.145) (width 0.5) (layer "F.Cu") (net 1))
