File: AL5801/testboard AL5801.kicad_sch (KiCad schematic)
At the start: 14 parts, among them J1 Conn_01x07_Pin, J3 Screw_Terminal_01x02, U1 AL5801W6-7, U2 INA169

Commit message: aanpassingen
Parts:
- R4: footprint Resistor_SMD:R_0805_2012Metric_Pad1.20x1.40mm_HandSolder -> Resistor_SMD:R_2512_6332Metric_Pad1.40x3.35mm_HandSolder
Connections:
- net enable  is gone; now on net enable: R4.2, U2.3 (+)
Changed lines of the file:
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@@
     (effects (font (size 1.27 1.27)) (justify right bottom))
+  )
+  (label "enable" (at 66.04 43.815 0) (fields_autoplaced)
+    (effects (font (size 1.27 1.27)) (justify left bottom))
   )
   (label "enable" (at 45.72 57.785 0) (fields_autoplaced)
@@
   (label "sda" (at 30.48 78.105 180) (fields_autoplaced)
     (effects (font (size 1.27 1.27)) (justify right bottom))
-  )
-  (label "enable " (at 66.04 43.815 0) (fields_autoplaced)
-    (effects (font (size 1.27 1.27)) (justify left bottom))
   )
   (label "led-" (at 114.935 46.355 0) (fields_autoplaced)
@@
       (effects (font (size 1.27 1.27)) (justify right))
     )
-    (property "Footprint" "Resistor_SMD:R_0805_2012Metric_Pad1.20x1.40mm_HandSolder" (at 80.01 46.355 0)
-      (effects (font (size 1.27 1.27)) hide)
-    )
+    (property "Footprint" "Resistor_SMD:R_2512_6332Metric_Pad1.40x3.35mm_HandSolder" (at 80.01 46.355 0)
+      (effects (font (size 1.27 1.27)) hide)
+    )

Commit message: ok
Connections:
- net enable renamed V_{in+}
Changed lines of the file:
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@@
     (effects (font (size 1.27 1.27)) (justify right bottom))
   )
-  (label "enable" (at 66.04 43.815 0) (fields_autoplaced)
+  (label "V_{in+}" (at 66.04 43.815 0) (fields_autoplaced)
     (effects (font (size 1.27 1.27)) (justify left bottom))
   )
-  (label "enable" (at 45.72 57.785 0) (fields_autoplaced)
+  (label "V_{in+}" (at 45.72 57.785 0) (fields_autoplaced)
     (effects (font (size 1.27 1.27)) (justify left bottom))
   )
@@
     (effects (font (size 1.27 1.27)) (justify left bottom))
   )
-  (label "enable" (at 55.245 43.18 180) (fields_autoplaced)
+  (label "V_{in+}" (at 55.245 43.18 180) (fields_autoplaced)
     (effects (font (size 1.27 1.27)) (justify right bottom))
   )
